Commit message: Node created to approach target object, frontier exploration improved

File: Workspaces/nav_ws/src/leo_description/urdf/NUC.xacro (robot description, xacro)
@@ -4,7 +4,7 @@
   <link name="cuboid_object_link">
     <visual>
-      <origin xyz="0 0 -0.03"/>
+      <origin xyz="0 0 0.015"/>
       <geometry>
-        <box size="0.1 0.1 0.02"/>
+        <box size="0.117 0.101 0.0336"/>
       </geometry>
       <material name="cuboid_material">
@@ -13,7 +13,7 @@
     </visual>
     <collision>
-      <origin xyz="0 0 -0.03"/>
+      <origin xyz="0 0 0.015"/>
       <geometry>
-        <box size="0.1 0.1 0.02"/>
+        <box size="0.117 0.101 0.0336"/>
       </geometry>
     </collision>
@@ -26,5 +26,5 @@
   <!-- Cuboid attached to rover -->
   <joint name="cuboid_object_joint" type="fixed">
-    <origin xyz="-0.1225 0 0.085" rpy="0 0 0"/>
+    <origin xyz="-0.090 0 0.0095" rpy="0 0 0"/>
     <parent link="base_link"/>
     <child link="cuboid_object_link"/>

File: Workspaces/nav_ws/src/leo_description/urdf/leo_sim.urdf.xacro (robot description, xacro)
@@ -8,4 +8,5 @@
   <xacro:include filename="lidar.xacro"/>
   <xacro:include filename="NUC.xacro"/>
+  <xacro:include filename="depth_camera.xacro"/>
   <xacro:leo_sim robot_ns="$(arg robot_ns)"
                  fixed="$(arg fixed)"

File: Workspaces/nav_ws/src/leo_description/urdf/lidar.xacro (robot description, xacro)
@@ -2,5 +2,5 @@
 <robot>
   <joint name="rplidar_joint" type="fixed"> #  <!--Specifying fixed joint -->
-    <origin xyz="0.0775 0 0.05"/> <!--Defining position w.r.t parent link (body_link)   -->
+    <origin xyz="0.0841 0 0.0115"/> <!--Defining position w.r.t parent link (body_link)   -->
     <parent link="base_link"/>  <!-- # What the lidar is being attached to -->
     <child link="rplidar_link"/> <!-- # The lidar -->
@@ -10,7 +10,7 @@
     <!--Visual properties of lidar's base-->
     <visual>
-      <origin xyz="0 0 0.0085"/>
+      <origin xyz="0 0 0.0015"/>
       <geometry>
-        <box size="0.080 0.087 0.017"/>
+        <box size="0.080 0.087 0.0185"/>
       </geometry>
       <material name="support">
@@ -20,5 +20,5 @@
     <!--Visual properties of lidar's main body -->
     <visual>
-      <origin xyz="0 0 0.034"/>
+      <origin xyz="0 0 0.0263"/>
       <geometry>
         <cylinder radius="0.038" length="0.041"/>
@@ -30,12 +30,12 @@
     <!-- Collision properties of lidar's base -->
     <collision>
-      <origin xyz="0 0 0.0085"/>
+      <origin xyz="0 0 0.0015"/>
       <geometry>
-        <box size="0.080 0.087 0.017"/>
+        <box size="0.080 0.087 0.0185"/>
       </geometry>
     </collision>
     <!-- Collision properties of lidar's main body -->
     <collision>
-      <origin xyz="0 0 0.034"/>
+      <origin xyz="0 0 0.0263"/>
       <geometry>
         <cylinder radius="0.038" length="0.041"/>
@@ -53,5 +53,5 @@
   <gazebo reference = "rplidar_link">
     <sensor name = "base_scan" type = "gpu_lidar">
-      <pose relative_to='rplidar_link'> 0 0 0 0 0 0 </pose>
+      <pose relative_to='rplidar_link'> 0 0 0.035 0 0 0 </pose>
       <topic>scan</topic>
       <gz_frame_id>rplidar_link</gz_frame_id>
