Commit message: 30_apr_push

File: Workspaces/nav_ws/src/leo_description/urdf/depth_camera.xacro (robot description, xacro)
@@ -32,5 +32,5 @@
   <!-- ====================== MOUNT JOINT ====================== -->
   <joint name="realsense_mount_joint" type="fixed">
-    <origin xyz="0.10 0 0.1" rpy="0 0 0"/>
+    <origin xyz="0.17 0.0 0.0225" rpy="0 0 0"/>
     <parent link="base_link"/>  <!-- change to your robot’s base link -->
     <child link="realsense_link"/>

File: Workspaces/nav_ws/src/leo_description/urdf/leo_sim.urdf.xacro (robot description, xacro)
@@ -9,4 +9,7 @@
   <xacro:include filename="NUC.xacro"/>
   <xacro:include filename="depth_camera.xacro"/>
+  <xacro:include filename="model.xacro"/>
+  <xacro:include filename="storage_box.xacro"/>
+  <xacro:include filename="tracking_cams.xacro"/>
   <xacro:leo_sim robot_ns="$(arg robot_ns)"
                  fixed="$(arg fixed)"

File: Workspaces/nav_ws/src/leo_description/urdf/lidar.xacro (robot description, xacro)
@@ -1,57 +1,41 @@
 <?xml version="1.0"?>
-<robot>
-  <joint name="rplidar_joint" type="fixed"> #  <!--Specifying fixed joint -->
-    <origin xyz="0.0841 0 0.0115"/> <!--Defining position w.r.t parent link (body_link)   -->
-    <parent link="base_link"/>  <!-- # What the lidar is being attached to -->
-    <child link="rplidar_link"/> <!-- # The lidar -->
+<robot xmlns:xacro="http://www.ros.org/wiki/xacro">
+  <!-- ============================
+       LIDAR MOUNTING JOINT
+  ============================= -->
+  <joint name="rplidar_joint" type="fixed">
+    <!-- Position of lidar relative to rover base_link -->
+    <origin xyz="${84.806/1000} 0 ${15/1000}" rpy="0 0 0"/>
+    <parent link="base_link"/>
+    <child link="rplidar_link"/>
   </joint>
-  <!--Defining visual and collision properties of lidar (could add 3D model of lidar) -->
-  <link name="rplidar_link"> <!--Defining lidar link name  -->
-    <!--Visual properties of lidar's base-->
+  <!-- ============================
+       LIDAR LINK + STL GEOMETRY
+  ============================= -->
+  <link name="rplidar_link">
+    <!-- Visual model -->
     <visual>
-      <origin xyz="0 0 0.0015"/>
+      <origin xyz="0 0 0" rpy="0 0 0"/>
       <geometry>
-        <box size="0.080 0.087 0.0185"/>
+        <mesh filename="package://leo_description/models/lidar_holder.stl"
+              scale="0.001 0.001 0.001"/>
       </geometry>
-      <material name="support">
-        <color rgba="0.5 0.5 0.5 1.0"/>
-      </material>
     </visual>
-    <!--Visual properties of lidar's main body -->
-    <visual>
-      <origin xyz="0 0 0.0263"/>
+    <!-- Collision model -->
+    <collision>
+      <origin xyz="0 0 0" rpy="0 0 0"/>
       <geometry>
-        <cylinder radius="0.038" length="0.041"/>
-      </geometry>
-      <material name="lidar">
-        <color rgba="1.0 0.0 0.0 0.7"/>
-      </material>
-    </visual>
-    <!-- Collision properties of lidar's base -->
-    <collision>
-      <origin xyz="0 0 0.0015"/>
-      <geometry>
-        <box size="0.080 0.087 0.0185"/>
-      </geometry>
-    </collision>
-    <!-- Collision properties of lidar's main body -->
-    <collision>
-      <origin xyz="0 0 0.0263"/>
-      <geometry>
-        <cylinder radius="0.038" length="0.041"/>
+        <mesh filename="package://leo_description/models/lidar_holder.stl"
+              scale="0.001 0.001 0.001"/>
       </geometry>
     </collision>
   </link>
-  <!--<gazebo>
-    <plugin
-      filename="gz-sim-sensors-system"
-      name="gz::sim::systems::Sensors">
-      <frame_id>rplidar_link</frame_id>
-      <render_engine>ogre2</render_engine>
-    </plugin>
-  </gazebo>-->
-  <gazebo reference = "rplidar_link">
-    <sensor name = "base_scan" type = "gpu_lidar">
-      <pose relative_to='rplidar_link'> 0 0 0.035 0 0 0 </pose>
+  <!-- ============================
+       GAZEBO GPU LIDAR SENSOR
+  ============================= -->
+  <gazebo reference="rplidar_link">
+    <sensor name="base_scan" type="gpu_lidar">
+      <!-- Sensor pose relative to rplidar_link -->
+      <pose relative_to="rplidar_link">0 0 0.0495 0 0 0</pose>
       <topic>scan</topic>
       <gz_frame_id>rplidar_link</gz_frame_id>
@@ -67,5 +51,5 @@
         </scan>
         <range>
-          <min>0.03</min>
+          <min>0.2225</min>
           <max>12</max>
           <resolution>0.005</resolution>
@@ -76,9 +60,12 @@
     </sensor>
   </gazebo>
-<link name="leo_rover/base_footprint/base_scan"/>
-<joint name="scan_tf_joint" type="fixed">
-  <origin xyz="0 0 0.483" rpy="0 0 ${-pi/2}"/>
-  <parent link="rplidar_link"/>
-  <child link="leo_rover/base_footprint/base_scan"/>
-</joint>
+  <!-- ============================
+       TF LINK FOR SCAN FRAME
+  ============================= -->
+  <link name="leo_rover/base_footprint/base_scan"/>
+  <joint name="scan_tf_joint" type="fixed">
+    <origin xyz="0 0 ${49.5/1000}" rpy="0 0 ${-pi/2}"/>
+    <parent link="rplidar_link"/>
+    <child link="leo_rover/base_footprint/base_scan"/>
+  </joint>
 </robot>
